Commit message: fixed a bug!

File: scout_gazebo/urdf/base.xacro (robot description, xacro)
@@ -59,10 +59,10 @@
         </collision>
     </link>
-    <!-- <link name="base_footprint"/>
+    <link name="base_footprint"/>
     <joint name="base_footprint_joint" type="fixed">
         <origin xyz="0 0 0" rpy="0 0 0" />
-        <parent link="base_footprint" />
-        <child link="base_link" />
-    </joint> -->
+        <parent link="base_link" />
+        <child link="base_footprint" />
+    </joint>
     <link name="inertial_link">
         <inertial>
